Commit message: push xml/copypaste

File: urdf/digit-v3.urdf (robot description, URDF)
Before this commit: robot digit, 37 links, 36 joints
Links:
- removed link left_achilles_rod
- removed link left_elbow
- removed link left_heel_spring
- removed link left_hip_pitch
- removed link left_hip_roll
- removed link left_hip_yaw
- removed link left_knee
- removed link left_shin
- removed link left_shoulder_pitch
- removed link left_shoulder_roll
- removed link left_shoulder_yaw
- removed link left_tarsus
- removed link left_toe_A
- removed link left_toe_A_rod
- removed link left_toe_B
- removed link left_toe_B_rod
- removed link left_toe_pitch
- removed link left_toe_roll
- removed link right_achilles_rod
- removed link right_elbow
- removed link right_heel_spring
- removed link right_hip_pitch
- removed link right_hip_roll
- removed link right_hip_yaw
- removed link right_knee
- removed link right_shin
- removed link right_shoulder_pitch
- removed link right_shoulder_roll
- removed link right_shoulder_yaw
- removed link right_tarsus
- removed link right_toe_A
- removed link right_toe_A_rod
- removed link right_toe_B
- removed link right_toe_B_rod
- removed link right_toe_pitch
- removed link right_toe_roll
- added link left-leg/hip-roll, mass 0.915088; collision mesh filename=package://urdf/stl/leg-v3/hip-yaw-housing.stl; visual mesh filename=package://urdf/stl/leg-v3/hip-yaw-housing.stl
- link torso: geometry collision mesh filename=package://urdf/stl/arm-v3/link-0.stl; collision mesh filename=package://urdf/stl/arm-v3/link-0.stl
Joints:
- removed joint elbow_joint_left
- removed joint elbow_joint_right
- removed joint hip_abduction_right
- removed joint hip_flexion_left
- removed joint hip_flexion_right
- removed joint hip_pitch_achilles_rod_left
- removed joint hip_pitch_achilles_rod_right
- removed joint hip_rotation_left
- removed joint hip_rotation_right
- removed joint knee_joint_left
- removed joint knee_joint_right
- removed joint knee_to_shin_left
- removed joint knee_to_shin_right
- removed joint shin_to_tarsus_left
- removed joint shin_to_tarsus_right
- removed joint shoulder_pitch_joint_left
- removed joint shoulder_pitch_joint_right
- removed joint shoulder_roll_joint_left
- removed joint shoulder_roll_joint_right
- removed joint shoulder_yaw_joint_left
- removed joint shoulder_yaw_joint_right
- removed joint tarsus_heel_spring_left
- removed joint tarsus_heel_spring_right
- removed joint tarsus_toe_A_left
- removed joint tarsus_toe_A_right
- removed joint tarsus_toe_B_left
- removed joint tarsus_toe_B_right
- removed joint toe_A_toe_A_rod_left
- removed joint toe_A_toe_A_rod_right
- removed joint toe_B_toe_B_rod_left
- removed joint toe_B_toe_B_rod_right
- removed joint toe_pitch_joint_left
- removed joint toe_pitch_joint_right
- removed joint toe_roll_joint_left
- removed joint toe_roll_joint_right
- joint hip_abduction_left: child left_hip_roll -> left-leg/hip-roll

Commit message: parameter tuning for back drop of digit

File: urdf/digit-v3.urdf (robot description, URDF)
Before this commit: robot digit, 2 links, 1 joints
Links:
- removed link left-leg/hip-roll
- added link left_A2, mass 0.; collision sphere radius=0.0; visual sphere radius=0.0
- added link left_B2, mass 0.; collision sphere radius=0.0; visual sphere radius=0.0
- added link left_ach2, mass 0.; collision sphere radius=0.0; visual sphere radius=0.0
- added link left_achilles_rod, mass 0.178148; collision mesh filename=package://urdf/stl/leg-v3/achilles-rod.stl; visual mesh filename=package://urdf/stl/leg-v3/achilles-rod.stl
- added link left_elbow, mass 0.550582; collision mesh filename=package://urdf/stl/arm-v3/link-4.stl; visual mesh filename=package://urdf/stl/arm-v3/link-4.stl
- added link left_heel_spring, mass 0.230018; collision mesh filename=package://urdf/stl/leg-v3/heel-spring.stl; visual mesh filename=package://urdf/stl/leg-v3/heel-spring.stl
- added link left_hip_pitch, mass 6.244279; collision mesh filename=package://urdf/stl/leg-v3/hip-pitch.stl; visual mesh filename=package://urdf/stl/leg-v3/hip-pitch.stl
- added link left_hip_roll, mass 0.915088; collision mesh filename=package://urdf/stl/leg-v3/hip-yaw-housing.stl; visual mesh filename=package://urdf/stl/leg-v3/hip-yaw-housing.stl
- added link left_hip_yaw, mass 0.818753; collision mesh filename=package://urdf/stl/leg-v3/hip-pitch-housing.stl; visual mesh filename=package://urdf/stl/leg-v3/hip-pitch-housing.stl
- added link left_knee, mass 1.227077; collision mesh filename=package://urdf/stl/leg-v3/knee.stl; visual mesh filename=package://urdf/stl/leg-v3/knee.stl
- added link left_shin, mass 0.895793; collision mesh filename=package://urdf/stl/leg-v3/shin.stl; visual mesh filename=package://urdf/stl/leg-v3/shin.stl
- added link left_shoulder_pitch, mass 1.440357; collision mesh filename=package://urdf/stl/arm-v3/link-2.stl; visual mesh filename=package://urdf/stl/arm-v3/link-2.stl
- added link left_shoulder_roll, mass 0.535396; collision mesh filename=package://urdf/stl/arm-v3/link-1.stl; visual mesh filename=package://urdf/stl/arm-v3/link-1.stl
- added link left_shoulder_yaw, mass 1.065387; collision mesh filename=package://urdf/stl/arm-v3/link-3.stl; visual mesh filename=package://urdf/stl/arm-v3/link-3.stl
- added link left_tarsus, mass 1.322865; collision mesh filename=package://urdf/stl/leg-v3/tarsus.stl; visual mesh filename=package://urdf/stl/leg-v3/tarsus.stl
- added link left_toe_A, mass 0.139557; collision mesh filename=package://urdf/stl/leg-v3/toe-output.stl; visual mesh filename=package://urdf/stl/leg-v3/toe-output.stl
- added link left_toe_A_rod, mass 0.090983; collision mesh filename=package://urdf/stl/leg-v3/toe-a-rod.stl; visual mesh filename=package://urdf/stl/leg-v3/toe-a-rod.stl
- added link left_toe_B, mass 0.139557; collision mesh filename=package://urdf/stl/leg-v3/toe-output.stl; visual mesh filename=package://urdf/stl/leg-v3/toe-output.stl
- added link left_toe_B_rod, mass 0.079507; collision mesh filename=package://urdf/stl/leg-v3/toe-a-rod.stl; visual mesh filename=package://urdf/stl/leg-v3/toe-a-rod.stl
- added link left_toe_pitch, mass 0.043881; collision mesh filename=package://urdf/stl/leg-v3/toe-pitch.stl; visual mesh filename=package://urdf/stl/leg-v3/toe-pitch.stl
- added link left_toe_roll, mass 0.531283; collision mesh filename=package://urdf/stl/leg-v3/toe-roll.stl; visual mesh filename=package://urdf/stl/leg-v3/toe-roll.stl
- added link right_A2, mass 0.; collision sphere radius=0.0; visual sphere radius=0.0
- added link right_B2, mass 0.; collision sphere radius=0.0; visual sphere radius=0.0
- added link right_ach2, mass 0.; collision sphere radius=0.0; visual sphere radius=0.0
- added link right_achilles_rod, mass 0.178148; collision mesh filename=package://urdf/stl/leg-v3/achilles-rod.stl scale=1 -1 1; visual mesh filename=package://urdf/stl/leg-v3/achilles-rod.stl scale=1 -1 1
- added link right_elbow, mass 0.550582; collision mesh filename=package://urdf/stl/arm-v3/link-4.stl scale=1 -1 1; visual mesh filename=package://urdf/stl/arm-v3/link-4.stl scale=1 -1 1
- added link right_heel_spring, mass 0.230018; collision mesh filename=package://urdf/stl/leg-v3/heel-spring.stl scale=1 -1 1; visual mesh filename=package://urdf/stl/leg-v3/heel-spring.stl scale=1 -1 1
- added link right_hip_pitch, mass 6.244279; collision mesh filename=package://urdf/stl/leg-v3/hip-pitch.stl scale=1 -1 1; visual mesh filename=package://urdf/stl/leg-v3/hip-pitch.stl scale=1 -1 1
- added link right_hip_roll, mass 0.915088; collision mesh filename=package://urdf/stl/leg-v3/hip-yaw-housing.stl scale=1 -1 1; visual mesh filename=package://urdf/stl/leg-v3/hip-yaw-housing.stl scale=1 -1 1
- added link right_hip_yaw, mass 0.818753; collision mesh filename=package://urdf/stl/leg-v3/hip-pitch-housing.stl scale=1 -1 1; visual mesh filename=package://urdf/stl/leg-v3/hip-pitch-housing.stl scale=1 -1 1
- added link right_knee, mass 1.227077; collision mesh filename=package://urdf/stl/leg-v3/knee.stl scale=1 -1 1; visual mesh filename=package://urdf/stl/leg-v3/knee.stl scale=1 -1 1
- added link right_shin, mass 0.895793; collision mesh filename=package://urdf/stl/leg-v3/shin.stl scale=1 -1 1; visual mesh filename=package://urdf/stl/leg-v3/shin.stl scale=1 -1 1
- added link right_shoulder_pitch, mass 1.440357; collision mesh filename=package://urdf/stl/arm-v3/link-2.stl scale=1 -1 1; visual mesh filename=package://urdf/stl/arm-v3/link-2.stl scale=1 -1 1
- added link right_shoulder_roll, mass 0.535396; collision mesh filename=package://urdf/stl/arm-v3/link-1.stl scale=1 -1 1; visual mesh filename=package://urdf/stl/arm-v3/link-1.stl scale=1 -1 1
- added link right_shoulder_yaw, mass 1.065387; collision mesh filename=package://urdf/stl/arm-v3/link-3.stl scale=1 -1 1; visual mesh filename=package://urdf/stl/arm-v3/link-3.stl scale=1 -1 1
- added link right_tarsus, mass 1.322865; collision mesh filename=package://urdf/stl/leg-v3/tarsus.stl scale=1 -1 1; visual mesh filename=package://urdf/stl/leg-v3/tarsus.stl scale=1 -1 1
- added link right_toe_A, mass 0.139557; collision mesh filename=package://urdf/stl/leg-v3/toe-output.stl scale=1 -1 1; visual mesh filename=package://urdf/stl/leg-v3/toe-output.stl scale=1 -1 1
- added link right_toe_A_rod, mass 0.090983; collision mesh filename=package://urdf/stl/leg-v3/toe-a-rod.stl scale=1 -1 1; visual mesh filename=package://urdf/stl/leg-v3/toe-a-rod.stl scale=1 -1 1
- added link right_toe_B, mass 0.139557; collision mesh filename=package://urdf/stl/leg-v3/toe-output.stl scale=1 -1 1; visual mesh filename=package://urdf/stl/leg-v3/toe-output.stl scale=1 -1 1
- added link right_toe_B_rod, mass 0.079507; collision mesh filename=package://urdf/stl/leg-v3/toe-b-rod.stl scale=1 -1 1; visual mesh filename=package://urdf/stl/leg-v3/toe-b-rod.stl scale=1 -1 1
- added link right_toe_pitch, mass 0.043881; collision mesh filename=package://urdf/stl/leg-v3/toe-pitch.stl scale=1 -1 1; visual mesh filename=package://urdf/stl/leg-v3/toe-pitch.stl scale=1 -1 1
- added link right_toe_roll, mass 0.531283; collision mesh filename=package://urdf/stl/leg-v3/toe-roll.stl scale=1 -1 1; visual mesh filename=package://urdf/stl/leg-v3/toe-roll.stl scale=1 -1 1
Joints:
- removed joint hip_abduction_left
- added joint left_A2: type revolute, parent left_toe_A_rod, child left_A2, origin xyz=0 0 0 rpy=0 0 0, axis 0 1 0, limit lower=-1.7453 upper=1.7453 effort=0.9 velocity=11.5
- added joint left_B2: type revolute, parent left_toe_B_rod, child left_B2, origin xyz=0 0 0 rpy=0 0 0, axis 0 1 0, limit lower=-1.7453 upper=1.7453 effort=0.9 velocity=11.5
- added joint left_ach2: type revolute, parent left_achilles_rod, child left_ach2, origin xyz=0 0 0 rpy=0 0 0, axis 0 1 0, limit lower=-1.7453 upper=1.7453 effort=0.9 velocity=11.5
- added joint left_achilles_rod: type revolute, parent left_hip_pitch, child left_achilles_rod, origin xyz=0 0 0.046 rpy=0.0714    0.09   -1.4359, axis 0 0 1, limit lower=-1.7453 upper=1.7453 effort=12.5 velocity=8.5085
- added joint left_elbow: type revolute, parent left_shoulder_yaw, child left_elbow, origin xyz=0 -0.0385 0.185 rpy=1.57079632679 -0.3926991 0, axis 0 0 1, limit lower=-1.3526 upper=1.3526 effort=1.4 velocity=12.5
- added joint left_heel_spring: type revolute, parent left_tarsus, child left_heel_spring, origin xyz=-0.01766 -0.029456 0.00104 rpy=0.0780    0.0056    2.7192, axis 0 0 1, limit lower=-0.1047 upper=0.1047 effort=12 velocity=11.5
- added joint left_hip_pitch: type revolute, parent left_hip_yaw, child left_hip_pitch, origin xyz=0 0.004 0.068 rpy=-1.57079632679 -0.785398163397 3.14159265359, axis 0 0 -1, limit lower=-1.0472 upper=1.57079632679 effort=12.5 velocity=8.5
- added joint left_hip_roll: type revolute, parent torso, child left_hip_roll, origin xyz=-0.001 0.091 0 rpy=1.57079632679 -1.1955506 -1.57079632679, axis 0 0 1, limit lower=-1.0472 upper=1.0472 effort=1.4 velocity=12.15
- added joint left_hip_yaw: type revolute, parent left_hip_roll, child left_hip_yaw, origin xyz=-0.0505 0 0.044 rpy=0 -1.57079632679 0, axis 0 0 1, limit lower=-0.698132 upper=0.698132 effort=1.4 velocity=12.15
- added joint left_knee: type revolute, parent left_hip_pitch, child left_knee, origin xyz=0.12 0 0.0045 rpy=0 0 -1.57079632679, axis 0 0 1, limit lower=-1.2392 upper=0.8727 effort=12.5 velocity=8.5085
- added joint left_shin: type revolute, parent left_knee, child left_shin, origin xyz=0.060677 0.047406 0 rpy=0 0 0, axis 0 0 1, limit lower=-0.35 upper=0.35 effort=0 velocity=10
- added joint left_shoulder_pitch: type revolute, parent left_shoulder_roll, child left_shoulder_pitch, origin xyz=-0.00317 -0.011055 0.0555 rpy=1.57079632679 0.785398163397 -0.2792527, axis 0 0 -1, limit lower=-2.5307 upper=2.5307 effort=1.4 velocity=12.5
- added joint left_shoulder_roll: type revolute, parent torso, child left_shoulder_roll, origin xyz=-0.001 0.12 0.4 rpy=-1.57079632679 -1.3962633 1.57079632679, axis 0 0 1, limit lower=-1.309 upper=1.309 effort=1.4 velocity=12.5
- added joint left_shoulder_yaw: type revolute, parent left_shoulder_pitch, child left_shoulder_yaw, origin xyz=0 -0.165 -0.1 rpy=1.57079632679 0 0, axis 0 0 1, limit lower=-1.7453 upper=1.7453 effort=1.4 velocity=10
- added joint left_tarsus: type revolute, parent left_shin, child left_tarsus, origin xyz=0.434759 0.02 0 rpy=0 0 1.7976891, axis 0 0 1, limit lower=-0.8779 upper=1.2497 effort=0 velocity=20
- added joint left_toe_A: type revolute, parent left_tarsus, child left_toe_A, origin xyz=0.059 -0.034 -0.0276 rpy=-3.1416         0    -1.5526, axis 0 0 1, limit lower=-0.8077 upper=0.7851 effort=0.9 velocity=11.5
- added joint left_toe_A_rod: type revolute, parent left_toe_A, child left_toe_A_rod, origin xyz=0.057 0 -0.008 rpy=0.0059    0.0374   -1.5437, axis 0 0 1, limit lower=-1.7453 upper=1.7453 effort=0.9 velocity=11.5
- added joint left_toe_B: type revolute, parent left_tarsus, child left_toe_B, origin xyz=0.111 -0.034 0.0276 rpy=0         0   -1.5526, axis 0 0 1, limit lower=-0.8010 upper=0.7950 effort=0.9 velocity=11.5
- added joint left_toe_B_rod: type revolute, parent left_toe_B, child left_toe_B_rod, origin xyz=0.057 0 -0.008 rpy=-0.0038   -0.0538    1.5418, axis 0 0 1, limit lower=-1.7453 upper=1.7453 effort=0.9 velocity=11.5
- added joint left_toe_pitch: type revolute, parent left_tarsus, child left_toe_pitch, origin xyz=0.408 -0.04 0 rpy=0 0 1.2523, axis 0 0 1, limit lower=-0.7679 upper=0.5934 effort=0.9 velocity=11.5
- added joint left_toe_roll: type revolute, parent left_toe_pitch, child left_toe_roll, origin xyz=0 0 0 rpy=0 1.570779 0, axis 0 0 1, limit lower=-0.6458 upper=0.5760 effort=0.9 velocity=11.5
- added joint right_A2: type revolute, parent right_toe_A_rod, child right_A2, origin xyz=0 0 0 rpy=0 0 0, axis 0 1 0, limit lower=-1.7453 upper=1.7453 effort=0.9 velocity=11.5
- added joint right_B2: type revolute, parent right_toe_B_rod, child right_B2, origin xyz=0 0 0 rpy=0 0 0, axis 0 1 0, limit lower=-1.7453 upper=1.7453 effort=0.9 velocity=11.5
- added joint right_ach2: type revolute, parent right_achilles_rod, child right_ach2, origin xyz=0 0 0 rpy=0 0 0, axis 0 1 0, limit lower=-1.7453 upper=1.7453 effort=0.9 velocity=11.5
- added joint right_achilles_rod: type revolute, parent right_hip_pitch, child right_achilles_rod, origin xyz=0 0 0.046 rpy=-0.0714    0.09    1.4359, axis 0 0 1, limit lower=-1.7453 upper=1.7453 effort=12.5 velocity=8.5085
- added joint right_elbow: type revolute, parent right_shoulder_yaw, child right_elbow, origin xyz=0 0.0385 0.185 rpy=-1.57079632679 -0.3926991 0, axis 0 0 1, limit lower=-1.3526 upper=1.3526 effort=1.4 velocity=12.5
- added joint right_heel_spring: type revolute, parent right_tarsus, child right_heel_spring, origin xyz=-0.01766 0.029456 0.00104 rpy=-0.0780    0.0056   -2.7192, axis 0 0 1, limit lower=-0.1047 upper=0.1047 effort=12 velocity=11.5
- added joint right_hip_pitch: type revolute, parent right_hip_yaw, child right_hip_pitch, origin xyz=0 -0.004 0.068 rpy=1.57079632679 -0.785398163397 -3.14159265359, axis 0 0 -1, limit lower=-1.57079632679 upper=1.0472 effort=12.5 velocity=8.5
- added joint right_hip_roll: type revolute, parent torso, child right_hip_roll, origin xyz=-0.001 -0.091 0 rpy=-1.57079632679 -1.1955506 1.57079632679, axis 0 0 1, limit lower=-1.0472 upper=1.0472 effort=1.4 velocity=12.15
- added joint right_hip_yaw: type revolute, parent right_hip_roll, child right_hip_yaw, origin xyz=-0.0505 0 0.044 rpy=0 -1.57079632679 0, axis 0 0 1, limit lower=-0.698132 upper=0.698132 effort=1.4 velocity=12.15
- added joint right_knee: type revolute, parent right_hip_pitch, child right_knee, origin xyz=0.12 0 0.0045 rpy=0 0 1.57079632679, axis 0 0 1, limit lower=-1.0193 upper=1.3963 effort=12.5 velocity=8.5085
- added joint right_shin: type revolute, parent right_knee, child right_shin, origin xyz=0.060677 -0.047406 0 rpy=0 0 0, axis 0 0 1, limit lower=-0.35 upper=0.35 effort=0 velocity=10
- added joint right_shoulder_pitch: type revolute, parent right_shoulder_roll, child right_shoulder_pitch, origin xyz=-0.00317 0.011055 0.0555 rpy=-1.57079632679 0.785398163397 0.2792527, axis 0 0 -1, limit lower=-2.5307 upper=2.5307 effort=1.4 velocity=12.5
- added joint right_shoulder_roll: type revolute, parent torso, child right_shoulder_roll, origin xyz=-0.001 -0.12 0.4 rpy=1.57079632679 -1.3962633 -1.57079632679, axis 0 0 1, limit lower=-1.309 upper=1.309 effort=1.4 velocity=12.5
- added joint right_shoulder_yaw: type revolute, parent right_shoulder_pitch, child right_shoulder_yaw, origin xyz=0 0.165 -0.1 rpy=-1.57079632679 0 0, axis 0 0 1, limit lower=-1.7453 upper=1.7453 effort=1.4 velocity=10
- added joint right_tarsus: type revolute, parent right_shin, child right_tarsus, origin xyz=0.434759 -0.02 0 rpy=0 0 -1.7976891, axis 0 0 1, limit lower=-1.2497 upper=0.8779 effort=0 velocity=20
- added joint right_toe_A: type revolute, parent right_tarsus, child right_toe_A, origin xyz=0.059 0.034 -0.0276 rpy=3.1416         0   1.5526, axis 0 0 1, limit lower=-0.7851 upper=0.8077 effort=0.9 velocity=11.5
- added joint right_toe_A_rod: type revolute, parent right_toe_A, child right_toe_A_rod, origin xyz=0.057 0 -0.008 rpy=-0.0059    0.0374    1.5437, axis 0 0 1, limit lower=-1.7453 upper=1.7453 effort=0.9 velocity=11.5
- added joint right_toe_B: type revolute, parent right_tarsus, child right_toe_B, origin xyz=0.111 0.034 0.0276 rpy=0         0    1.5526, axis 0 0 1, limit lower=-0.7950 upper=0.8010 effort=0.9 velocity=11.5
- added joint right_toe_B_rod: type revolute, parent right_toe_B, child right_toe_B_rod, origin xyz=0.057 0 -0.008 rpy=0.0038   -0.0538   -1.5418, axis 0 0 1, limit lower=-1.7453 upper=1.7453 effort=0.9 velocity=11.5
- added joint right_toe_pitch: type revolute, parent right_tarsus, child right_toe_pitch, origin xyz=0.408 0.04 0 rpy=0 0 -1.1956, axis 0 0 1, limit lower=-0.5934 upper=0.7679 effort=0.9 velocity=11.5
- added joint right_toe_roll: type revolute, parent right_toe_pitch, child right_toe_roll, origin xyz=0 0 0 rpy=0 1.57079632679 0, axis 0 0 1, limit lower=-0.5760 upper=0.6458 effort=0.9 velocity=11.5
